File: board/bigbutton/bigbutton.sch (KiCad schematic (older format))
At the start: 57 parts, among them J1 SWD, J2 USB_C_Receptacle_USB2.0, SW1 RESET, SW2 SMOL, SW3 LORGE, SW4 BOOT0, U1 STM32F303CBTx, U2 ATECC608A-SSHDA, U3 USBLC6-2, U4 SN74LV1T34DBV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

Commit message: Hopefully revision 2
Parts:
- C1, C10, C11, C12, C13, C14, C15, C16, C17, C18, C19, C2, C20, C21, C3, C4, C5, C6, C7, C8, C9: footprint Capacitor_SMD:C_0603_1608Metric_Pad1.05x0.95mm_HandSolder -> Capacitor_SMD:C_0603_1608Metric
- R1, R2, R3, R4, R5, R6: footprint Resistor_SMD:R_0603_1608Metric_Pad1.05x0.95mm_HandSolder -> Resistor_SMD:R_0603_1608Metric
- X1: footprint Crystal:Resonator-2Pin_W8.0mm_H3.5mm -> Crystal:Resonator-2Pin_W10.0mm_H5.0mm
Changed lines of the file:
@@
 F 0 "X1" V 2950 2350 50  0000 L CNN
 F 1 "16MHz" V 2850 2250 50  0000 L CNN
-F 2 "Crystal:Resonator-2Pin_W8.0mm_H3.5mm" H 2900 2600 50  0001 C CNN
+F 2 "Crystal:Resonator-2Pin_W10.0mm_H5.0mm" H 2900 2600 50  0001 C CNN
 F 3 "~" H 2900 2600 50  0001 C CNN
 	1    2900 2600
@@
 F 0 "C9" V 3000 2500 50  0000 R CNN
 F 1 "22pF" V 2900 2500 50  0000 R CNN
-F 2 "Capacitor_SMD:C_0603_1608Metric_Pad1.05x0.95mm_HandSolder" H 2800 2450 50  0001 C CNN
+F 2 "Capacitor_SMD:C_0603_1608Metric" H 2800 2450 50  0001 C CNN
 F 3 "~" H 2800 2450 50  0001 C CNN
 	1    2800 2450
@@
 F 0 "C10" V 2650 2800 50  0000 R CNN
 F 1 "22pF" V 2550 2800 50  0000 R CNN
-F 2 "Capacitor_SMD:C_0603_1608Metric_Pad1.05x0.95mm_HandSolder" H 2800 2750 50  0001 C CNN
+F 2 "Capacitor_SMD:C_0603_1608Metric" H 2800 2750 50  0001 C CNN
 F 3 "~" H 2800 2750 50  0001 C CNN
 	1    2800 2750
@@
 F 0 "R1" H 2959 946 50  0000 L CNN
 F 1 "1kΩ" H 2959 855 50  0000 L CNN
-F 2 "Resistor_SMD:R_0603_1608Metric_Pad1.05x0.95mm_HandSolder" H 2900 900 50  0001 C CNN
+F 2 "Resistor_SMD:R_0603_1608Metric" H 2900 900 50  0001 C CNN
 F 3 "~" H 2900 900 50  0001 C CNN
 	1    2900 900
@@
 F 0 "C7" H 2992 1646 50  0000 L CNN
 F 1 "100nF" H 2992 1555 50  0000 L CNN
-F 2 "Capacitor_SMD:C_0603_1608Metric_Pad1.05x0.95mm_HandSolder" H 2900 1600 50  0001 C CNN
+F 2 "Capacitor_SMD:C_0603_1608Metric" H 2900 1600 50  0001 C CNN
 F 3 "~" H 2900 1600 50  0001 C CNN
 	1    2900 1600
@@
 F 0 "R5" V 2400 5850 50  0000 L CNN
 F 1 "5.1kΩ" V 2400 5600 50  0000 L CNN
-F 2 "Resistor_SMD:R_0603_1608Metric_Pad1.05x0.95mm_HandSolder" H 2500 5800 50  0001 C CNN
+F 2 "Resistor_SMD:R_0603_1608Metric" H 2500 5800 50  0001 C CNN
 F 3 "~" H 2500 5800 50  0001 C CNN
 	1    2500 5800
@@
 F 0 "R4" V 2600 5750 50  0000 L CNN
 F 1 "5.1kΩ" V 2600 5500 50  0000 L CNN
-F 2 "Resistor_SMD:R_0603_1608Metric_Pad1.05x0.95mm_HandSolder" H 2500 5700 50  0001 C CNN
+F 2 "Resistor_SMD:R_0603_1608Metric" H 2500 5700 50  0001 C CNN
 F 3 "~" H 2500 5700 50  0001 C CNN
 	1    2500 5700
@@
 F 0 "C8" H 3800 1800 50  0000 L CNN
 F 1 "100nF" H 3700 1700 50  0000 L CNN
-F 2 "Capacitor_SMD:C_0603_1608Metric_Pad1.05x0.95mm_HandSolder" H 4000 1750 50  0001 C CNN
+F 2 "Capacitor_SMD:C_0603_1608Metric" H 4000 1750 50  0001 C CNN
 F 3 "~" H 4000 1750 50  0001 C CNN
 	1    4000 1750
@@
 F 0 "C11" H 800 3900 50  0000 L CNN
 F 1 "100nF" H 700 3800 50  0000 L CNN
-F 2 "Capacitor_SMD:C_0603_1608Metric_Pad1.05x0.95mm_HandSolder" H 1000 3850 50  0001 C CNN
+F 2 "Capacitor_SMD:C_0603_1608Metric" H 1000 3850 50  0001 C CNN
 F 3 "~" H 1000 3850 50  0001 C CNN
 	1    1000 3850
@@
 F 0 "R2" V 1804 4250 50  0000 C CNN
 F 1 "10kΩ" V 1895 4250 50  0000 C CNN
-F 2 "Resistor_SMD:R_0603_1608Metric_Pad1.05x0.95mm_HandSolder" H 2000 4250 50  0001 C CNN
+F 2 "Resistor_SMD:R_0603_1608Metric" H 2000 4250 50  0001 C CNN
 F 3 "~" H 2000 4250 50  0001 C CNN
 	1    2000 4250
@@
 F 0 "R3" V 2200 4450 50  0000 C CNN
 F 1 "10kΩ" V 2100 4450 50  0000 C CNN
-F 2 "Resistor_SMD:R_0603_1608Metric_Pad1.05x0.95mm_HandSolder" H 2000 4450 50  0001 C CNN
+F 2 "Resistor_SMD:R_0603_1608Metric" H 2000 4450 50  0001 C CNN
 F 3 "~" H 2000 4450 50  0001 C CNN
 	1    2000 4450
@@
 F 0 "C1" H 5600 950 50  0000 L CNN
 F 1 "100nF" H 5600 850 50  0000 L CNN
-F 2 "Capacitor_SMD:C_0603_1608Metric_Pad1.05x0.95mm_HandSolder" H 5500 900 50  0001 C CNN
+F 2 "Capacitor_SMD:C_0603_1608Metric" H 5500 900 50  0001 C CNN
 F 3 "~" H 5500 900 50  0001 C CNN
 	1    5500 900
@@
 F 0 "C2" H 6000 950 50  0000 L CNN
 F 1 "100nF" H 6000 850 50  0000 L CNN
-F 2 "Capacitor_SMD:C_0603_1608Metric_Pad1.05x0.95mm_HandSolder" H 5900 900 50  0001 C CNN
+F 2 "Capacitor_SMD:C_0603_1608Metric" H 5900 900 50  0001 C CNN
 F 3 "~" H 5900 900 50  0001 C CNN
 	1    5900 900
@@
 F 0 "C3" H 6400 950 50  0000 L CNN
 F 1 "100nF" H 6400 850 50  0000 L CNN
-F 2 "Capacitor_SMD:C_0603_1608Metric_Pad1.05x0.95mm_HandSolder" H 6300 900 50  0001 C CNN
+F 2 "Capacitor_SMD:C_0603_1608Metric" H 6300 900 50  0001 C CNN
 F 3 "~" H 6300 900 50  0001 C CNN
 	1    6300 900
@@
 F 0 "C6" H 7592 946 50  0000 L CNN
 F 1 "10nF" H 7592 855 50  0000 L CNN
-F 2 "Capacitor_SMD:C_0603_1608Metric_Pad1.05x0.95mm_HandSolder" H 7500 900 50  0001 C CNN
+F 2 "Capacitor_SMD:C_0603_1608Metric" H 7500 900 50  0001 C CNN
 F 3 "~" H 7500 900 50  0001 C CNN
 	1    7500 900
@@
 F 0 "C5" H 7288 946 50  0000 L CNN
 F 1 "1µF" H 7288 855 50  0000 L CNN
-F 2 "Capacitor_SMD:C_0603_1608Metric_Pad1.05x0.95mm_HandSolder" H 7200 900 50  0001 C CNN
+F 2 "Capacitor_SMD:C_0603_1608Metric" H 7200 900 50  0001 C CNN
 F 3 "~" H 7200 900 50  0001 C CNN
 	1    7200 900
@@
 F 0 "C4" H 6788 946 50  0000 L CNN
 F 1 "4.7µF" H 6788 855 50  0000 L CNN
-F 2 "Capacitor_SMD:C_0603_1608Metric_Pad1.05x0.95mm_HandSolder" H 6700 900 50  0001 C CNN
+F 2 "Capacitor_SMD:C_0603_1608Metric" H 6700 900 50  0001 C CNN
 F 3 "~" H 6700 900 50  0001 C CNN
 	1    6700 900
@@
 F 0 "C12" H 6700 1850 50  0000 L CNN
 F 1 "100nF" H 6550 1750 50  0000 L CNN
-F 2 "Capacitor_SMD:C_0603_1608Metric_Pad1.05x0.95mm_HandSolder" H 6900 1800 50  0001 C CNN
+F 2 "Capacitor_SMD:C_0603_1608Metric" H 6900 1800 50  0001 C CNN
 F 3 "~" H 6900 1800 50  0001 C CNN
 	1    6900 1800
@@
 F 0 "C13" H 7700 1850 50  0000 L CNN
 F 1 "100nF" H 7550 1750 50  0000 L CNN
-F 2 "Capacitor_SMD:C_0603_1608Metric_Pad1.05x0.95mm_HandSolder" H 7900 1800 50  0001 C CNN
+F 2 "Capacitor_SMD:C_0603_1608Metric" H 7900 1800 50  0001 C CNN
 F 3 "~" H 7900 1800 50  0001 C CNN
 	1    7900 1800
@@
 F 0 "C14" H 8700 1850 50  0000 L CNN
 F 1 "100nF" H 8550 1750 50  0000 L CNN
-F 2 "Capacitor_SMD:C_0603_1608Metric_Pad1.05x0.95mm_HandSolder" H 8900 1800 50  0001 C CNN
+F 2 "Capacitor_SMD:C_0603_1608Metric" H 8900 1800 50  0001 C CNN
 F 3 "~" H 8900 1800 50  0001 C CNN
 	1    8900 1800
@@
 F 0 "C15" H 9700 1850 50  0000 L CNN
 F 1 "100nF" H 9550 1750 50  0000 L CNN
-F 2 "Capacitor_SMD:C_0603_1608Metric_Pad1.05x0.95mm_HandSolder" H 9900 1800 50  0001 C CNN
+F 2 "Capacitor_SMD:C_0603_1608Metric" H 9900 1800 50  0001 C CNN
 F 3 "~" H 9900 1800 50  0001 C CNN
 	1    9900 1800
@@
 F 0 "C16" H 6700 3200 50  0000 L CNN
 F 1 "100nF" H 6550 3100 50  0000 L CNN
-F 2 "Capacitor_SMD:C_0603_1608Metric_Pad1.05x0.95mm_HandSolder" H 6900 3150 50  0001 C CNN
+F 2 "Capacitor_SMD:C_0603_1608Metric" H 6900 3150 50  0001 C CNN
 F 3 "~" H 6900 3150 50  0001 C CNN
 	1    6900 3150
@@
 F 0 "C17" H 7700 3200 50  0000 L CNN
 F 1 "100nF" H 7550 3100 50  0000 L CNN
-F 2 "Capacitor_SMD:C_0603_1608Metric_Pad1.05x0.95mm_HandSolder" H 7900 3150 50  0001 C CNN
+F 2 "Capacitor_SMD:C_0603_1608Metric" H 7900 3150 50  0001 C CNN
 F 3 "~" H 7900 3150 50  0001 C CNN
 	1    7900 3150
@@
 F 0 "C18" H 8700 3200 50  0000 L CNN
 F 1 "100nF" H 8550 3100 50  0000 L CNN
-F 2 "Capacitor_SMD:C_0603_1608Metric_Pad1.05x0.95mm_HandSolder" H 8900 3150 50  0001 C CNN
+F 2 "Capacitor_SMD:C_0603_1608Metric" H 8900 3150 50  0001 C CNN
 F 3 "~" H 8900 3150 50  0001 C CNN
 	1    8900 3150
@@
 F 0 "C19" H 9700 3200 50  0000 L CNN
 F 1 "100nF" H 9550 3100 50  0000 L CNN
-F 2 "Capacitor_SMD:C_0603_1608Metric_Pad1.05x0.95mm_HandSolder" H 9900 3150 50  0001 C CNN
+F 2 "Capacitor_SMD:C_0603_1608Metric" H 9900 3150 50  0001 C CNN
 F 3 "~" H 9900 3150 50  0001 C CNN
 	1    9900 3150
@@
 F 0 "C20" H 4300 6550 50  0000 L CNN
 F 1 "1µF" H 4250 6450 50  0000 L CNN
-F 2 "Capacitor_SMD:C_0603_1608Metric_Pad1.05x0.95mm_HandSolder" H 4500 6500 50  0001 C CNN
+F 2 "Capacitor_SMD:C_0603_1608Metric" H 4500 6500 50  0001 C CNN
 F 3 "~" H 4500 6500 50  0001 C CNN
 	1    4500 6500
@@
 F 0 "C21" H 5792 6546 50  0000 L CNN
 F 1 "1µF" H 5792 6455 50  0000 L CNN
-F 2 "Capacitor_SMD:C_0603_1608Metric_Pad1.05x0.95mm_HandSolder" H 5700 6500 50  0001 C CNN
+F 2 "Capacitor_SMD:C_0603_1608Metric" H 5700 6500 50  0001 C CNN
 F 3 "~" H 5700 6500 50  0001 C CNN
 	1    5700 6500
@@
 F 0 "R6" H 1709 2896 50  0000 L CNN
 F 1 "10kΩ" H 1709 2805 50  0000 L CNN
-F 2 "Resistor_SMD:R_0603_1608Metric_Pad1.05x0.95mm_HandSolder" H 1650 2850 50  0001 C CNN
+F 2 "Resistor_SMD:R_0603_1608Metric" H 1650 2850 50  0001 C CNN
 F 3 "~" H 1650 2850 50  0001 C CNN
 	1    1650 2850
